File: pcb/semafor-b-panel.brd (EAGLE design)
At the start: 97 x 96 mm, 35 parts

Commit message: Add missing ground wire to PCB and update gerbers
Routing:
- net N$15: track 65.2 -> 73.2 mm
Changed lines of the file:
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@@
 <wire x1="43.5" y1="14.5" x2="43.5" y2="10" width="0.1524" layer="1"/>
 <wire x1="45" y1="16" x2="43.5" y2="14.5" width="0.1524" layer="1"/>
+<wire x1="44.77" y1="66" x2="44.77" y2="74" width="0.1524" layer="1"/>
 </signal>
 <signal name="N$16">
